Commit message: working lidar

File: mrsearch_IG_RL/assets/map.urdf (robot description, URDF)
Before this commit: robot walls, 17 links, 16 joints
Joints:
- joint center: origin xyz=0 -3 1 rpy=0 0 0 -> xyz=0 -2.95 1 rpy=0 0 0
- joint center_left_horiz: origin xyz=-5.975 2.475 1 rpy=0 0 0 -> xyz=-6 2.575 1 rpy=0 0 0
- joint center_left_vert: origin xyz=-7.975 -0.25 1 rpy=0 0 0 -> xyz=-8.025 -0.175 1 rpy=0 0 0
- joint center_left_vert_down: origin xyz=-3.975 0.5 1 rpy=0 0 0 -> xyz=-3.975 0.55 1 rpy=0 0 0
- joint center_right: origin xyz=4.55 -1.55 1 rpy=0 0 0 -> xyz=4.5 -1.475 1 rpy=0 0 0
- joint center_right_horiz: origin xyz=2.825 -0.125 1 rpy=0 0 0 -> xyz=2.75 0 1 rpy=0 0 0
- joint center_vert: origin xyz=-2.5 -1.25 1 rpy=0 0 0 -> xyz=-1.6 -1.175 1 rpy=0 0 0
- joint down: origin xyz=0 -5 1 rpy=0 0 0 -> xyz=0.05 -5 1 rpy=0 0 0
- joint right: origin xyz=10.05 0 1 rpy=0 0 0 -> xyz=10.1 0 1 rpy=0 0 0
- joint table: origin xyz=1.75 2 1 rpy=0 0 0 -> xyz=1.7 2.05 1 rpy=0 0 0
- joint table_left: origin xyz=-0.5 2.625 1 rpy=0 0 0 -> xyz=-0.55 2.675 1 rpy=0 0 0
- joint table_right: origin xyz=4 2.625 1 rpy=0 0 0 -> xyz=3.95 2.675 1 rpy=0 0 0
- joint up: origin xyz=0 5.05 1 rpy=0 0 0 -> xyz=0.05 5.05 1 rpy=0 0 0
- joint uright_horiz: origin xyz=8.5 -0.05 1 rpy=0 0 0 -> xyz=8.55 0 1 rpy=0 0 0
