Commit message: fixed path planning

File: mrsearch_IG_RL/assets/robot.urdf (robot description, URDF)
Before this commit: robot robot, 1 links, 0 joints
Links:
- link base_link: geometry collision box size=0.5 0.5 0.5; visual box size=0.5 0.5 0.5

File: mrsearch_IG_RL/assets/target.urdf (robot description, URDF)
Before this commit: robot target, 1 links, 0 joints
Links:
- link base_link: geometry collision box size=0.5 0.5 1; visual box size=0.5 0.5 1

Commit message: reward scaling

File: mrsearch_IG_RL/assets/robot.urdf (robot description, URDF)
Before this commit: robot robot, 1 links, 0 joints
Links:
- link base_link: geometry collision cylinder length=0.5 radius=0.25; visual cylinder length=0.5 radius=0.25
